File: PCB Rev 2/VolumetricDisplay.kicad_pcb (KiCad board)
At the start: 4 copper layers, 48.5 x 56 mm, 149 parts, among them J1 USB_C_Receptacle_USB2.0_16P, J2 Conn_ARM_SWD_TagConnect_TC2030, Q1 DMN32D2LDF, Q2 DMN32D2LDF, Q3 DMN32D2LDF, Q4 DMN32D2LDF, SW4 TS-1088-AR02016, SW5 TS-1088-AR02016, U2 NCP718xSN330, U3 RP2354B, U4 DRV8311S, U5 DRV5055A1xDBZxQ1, Y1 Abracon ABM8-272-T3

Commit message: PCB Trace Attempts
Attempted to connect some of the photodiodes within the matrix. Also added one via from F.cu to B.cu
Routing:
- net Net-(D1-K): track 0.00 -> 43.0 mm, vias 0 -> 1
- net LED5: track 0.00 -> 38.6 mm
- net LED6: track 0.00 -> 38.5 mm
- net LED7: track 0.00 -> 38.5 mm
- net LED4: track 0.00 -> 38.5 mm
- net LED2: track 0.00 -> 38.5 mm
- net LED1: track 0.00 -> 38.5 mm
- net LED0: track 0.12 -> 38.6 mm
- net LED3: track 0.00 -> 38.5 mm
Changed lines of the file:
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@@
+	)
+	(segment
+		(start 140.076 122.71)
+		(end 140.076 84.21)
+		(width 0.2)
+		(layer "F.Cu")
+		(net "LED4")
+	)
+	(segment
+		(start 151.076 122.67)
+		(end 151.076 84.12)
+		(width 0.2)
+		(layer "F.Cu")
+		(net "LED6")
+	)
+	(segment
+		(start 123.576 84.21)
+		(end 123.576 122.71)
+		(width 0.2)
+		(layer "F.Cu")
+		(net "LED1")
+	)
+	(segment
+		(start 118.076 84.21)
+		(end 118.076 122.71)
+		(width 0.2)
+		(layer "F.Cu")
+		(net "LED0")
 	)
 	(segment
@@
 	)
 	(segment
+		(start 129.076 122.71)
+		(end 129.076 84.21)
+		(width 0.2)
+		(layer "F.Cu")
+		(net "LED2")
+	)
+	(segment
+		(start 145.576 84.21)
+		(end 145.576 122.85)
+		(width 0.2)
+		(layer "F.Cu")
+		(net "LED5")
+	)
+	(segment
+		(start 134.576 84.21)
+		(end 134.576 122.66)
+		(width 0.2)
+		(layer "F.Cu")
+		(net "LED3")
+	)
+	(segment
+		(start 132.826 84.21)
+		(end 133.526 83.51)
+		(width 0.2)
+		(layer "F.Cu")
+		(net "Net-(D1-K)")
+	)
+	(segment
+		(start 143.826 84.21)
+		(end 144.526 83.51)
+		(width 0.2)
+		(layer "F.Cu")
+		(net "Net-(D1-K)")
+	)
+	(segment
+		(start 128.026 83.51)
+		(end 127.326 84.21)
+		(width 0.2)
+		(layer "F.Cu")
+		(net "Net-(D1-K)")
+	)
+	(segment
+		(start 121.826 84.21)
+		(end 122.526 83.51)
+		(width 0.2)
+		(layer "F.Cu")
+		(net "Net-(D1-K)")
+	)
+	(segment
+		(start 149.326 84.12)
+		(end 150.026 83.42)
+		(width 0.2)
+		(layer "F.Cu")
+		(net "Net-(D1-K)")
+	)
+	(segment
+		(start 150.026 83.42)
+		(end 154.036 83.42)
+		(width 0.2)
+		(layer "F.Cu")
+		(net "Net-(D1-K)")
+	)
+	(segment
+		(start 117.536 83)
+		(end 119 83)
+		(width 0.2)
+		(layer "F.Cu")
+		(net "Net-(D1-K)")
+	)
+	(segment
+		(start 132.126 83.51)
+		(end 128.026 83.51)
+		(width 0.2)
+		(layer "F.Cu")
+		(net "Net-(D1-K)")
+	)
+	(segment
+		(start 148.716 83.51)
+		(end 149.326 84.12)
+		(width 0.2)
+		(layer "F.Cu")
+		(net "Net-(D1-K)")
+	)
+	(segment
+		(start 143.126 83.51)
+		(end 143.826 84.21)
+		(width 0.2)
+		(layer "F.Cu")
+		(net "Net-(D1-K)")
+	)
+	(segment
+		(start 119 83)
+		(end 120.616 83)
+		(width 0.2)
+		(layer "F.Cu")
+		(net "Net-(D1-K)")
+	)
+	(segment
+		(start 122.526 83.51)
+		(end 126.626 83.51)
+		(width 0.2)
+		(layer "F.Cu")
+		(net "Net-(D1-K)")
+	)
+	(segment
+		(start 126.626 83.51)
+		(end 127.326 84.21)
+		(width 0.2)
+		(layer "F.Cu")
+		(net "Net-(D1-K)")
+	)
+	(segment
+		(start 144.526 83.51)
+		(end 148.716 83.51)
+		(width 0.2)
+		(layer "F.Cu")
+		(net "Net-(D1-K)")
+	)
+	(segment
+		(start 116.326 84.21)
+		(end 117.536 83)
+		(width 0.2)
+		(layer "F.Cu")
+		(net "Net-(D1-K)")
+	)
+	(segment
+		(start 138.326 84.21)
+		(end 139.026 83.51)
+		(width 0.2)
+		(layer "F.Cu")
+		(net "Net-(D1-K)")
+	)
+	(segment
+		(start 137.626 83.51)
+		(end 138.326 84.21)
+		(width 0.2)
+		(layer "F.Cu")
+		(net "Net-(D1-K)")
+	)
+	(segment
+		(start 154.036 83.42)
+		(end 154.826 84.21)
+		(width 0.2)
+		(layer "F.Cu")
+		(net "Net-(D1-K)")
+	)
+	(segment
+		(start 120.616 83)
+		(end 121.826 84.21)
+		(width 0.2)
+		(layer "F.Cu")
+		(net "Net-(D1-K)")
+	)
+	(segment
+		(start 133.526 83.51)
+		(end 137.626 83.51)
+		(width 0.2)
+		(layer "F.Cu")
+		(net "Net-(D1-K)")
+	)
+	(segment
+		(start 139.026 83.51)
+		(end 143.126 83.51)
+		(width 0.2)
+		(layer "F.Cu")
+		(net "Net-(D1-K)")
+	)
+	(segment
+		(start 132.826 84.21)
+		(end 132.126 83.51)
+		(width 0.2)
+		(layer "F.Cu")
+		(net "Net-(D1-K)")
+	)
+	(via
+		(at 119 83)
+		(size 0.6)
+		(drill 0.3)
+		(layers "F.Cu" "B.Cu")
+		(net "Net-(D1-K)")
+	)
+	(segment
+		(start 156.576 84.21)
+		(end 156.576 122.71)
+		(width 0.2)
+		(layer "F.Cu")
+		(net "LED7")
+	)
+	(segment
