File: PCB Rev 2/VolumetricDisplay.kicad_pcb (KiCad board)
At the start: 4 copper layers, 48.5 x 56 mm, 149 parts, among them J1 USB_C_Receptacle_USB2.0_16P, J2 Conn_ARM_SWD_TagConnect_TC2030, Q1 DMN32D2LDF, Q2 DMN32D2LDF, Q3 DMN32D2LDF, Q4 DMN32D2LDF, SW4 TS-1088-AR02016, SW5 TS-1088-AR02016, U2 NCP718xSN330, U3 RP2354B, U4 DRV8311S, U5 DRV5055A1xDBZxQ1, Y1 Abracon ABM8-272-T3

Commit message: added some more roughting and fills
Routing:
- net Net-(D12-K): track 0.00 -> 7.00 mm, vias 0 -> 2
- net Net-(D10-K): track 0.00 -> 6.93 mm, vias 0 -> 2
- net Net-(D11-K): track 0.00 -> 6.82 mm, vias 0 -> 2
- net GND: track 4.29 -> 6.99 mm
- net /MCU/VBUS: track 0.00 -> 2.70 mm
- net D_P: track 15.9 -> 17.6 mm
- net D_N: track 15.6 -> 17.3 mm
- added copper zone on B.Cu, net GND
- added copper zone on F.Cu, net GND
- added copper zone on In1.Cu, net GND

Commit message: I finished tracings. have lots of warnings and errors
Routing:
- net GND: track 6.99 -> 310.2 mm, vias 0 -> 32
- net Net-(U3-GPIO12): track 0.00 -> 178.3 mm, vias 0 -> 3
- net 5V: track 18.8 -> 155.4 mm, vias 5 -> 10
- net 3V3: track 2.08 -> 129.4 mm, vias 0 -> 8
- net LED9: track 0.00 -> 68.4 mm
- net Net-(U3-GPIO10): track 0.00 -> 65.7 mm
- net +1V1: track 0.00 -> 57.8 mm, vias 0 -> 8
- net Net-(D14-K): track 0.00 -> 56.2 mm, vias 0 -> 14
- net LED15: track 0.00 -> 55.2 mm, vias 0 -> 2
- net LED12: track 0.00 -> 55.0 mm, vias 0 -> 2
- net LED0: track 38.6 -> 92.2 mm, vias 0 -> 5
- net LED11: track 0.00 -> 52.6 mm
- net /MCU/QSPI_CS: track 0.00 -> 52.2 mm
- net LED10: track 0.00 -> 52.1 mm
- net Net-(D16-K): track 1.29 -> 51.1 mm, vias 1 -> 8
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
Commit message: Fixed a few warnings and errors
Parts:
- moved R99 0.09 mm to (131.5, 119.9)
Routing:
- net GND: track 310.2 -> 279.1 mm
- net 5V: track 155.4 -> 158.6 mm
- net LED5: track 67.0 -> 69.9 mm, vias 1 -> 3
- net LED12: track 55.0 -> 56.8 mm, vias 2 -> 4
- net Net-(D15-K): track 47.0 -> 48.8 mm, vias 9 -> 7
- net nRST: track 45.3 -> 46.8 mm
- net Net-(D11-K): track 38.8 -> 37.4 mm
- net Net-(U3-GPIO7): track 38.5 -> 37.1 mm
- net 3V3: track 129.4 -> 130.4 mm, vias 8 -> 7
- net SPI_MOSI: track 4.43 -> 5.30 mm
- net LED3: track 60.9 -> 60.8 mm, vias 8 -> 7
- net Net-(D16-K): vias 8 -> 7
- net Net-(U3-GPIO5): vias 3 -> 2
